File: pcb_v0/pcb_v0.kicad_sch (KiCad schematic)
At the start: 28 parts, among them J1 Screw_Terminal_01x03, Q1 Q_NMOS_GDS, U1 ATtiny2313-20P, U10 74141, U2 74141, U3 74141, U4 74141, U5 74LS377, U6 74141, U7 74141, U8 74LS377, U9 74LS377

Commit message: save
Connections:
- net at U7.3 (A): now also U9.12 (Q4); no longer U9.2 (Q0)
- net at U7.4 (D): now also U9.19 (Q7); no longer U9.9 (Q3)
- net at U7.6 (B): now also U9.15 (Q5); no longer U9.5 (Q1)
- net at U7.7 (C): now also U9.16 (Q6); no longer U9.6 (Q2)
- net at U10.3 (A): now also U9.2 (Q0); no longer U9.12 (Q4)
- net at U10.4 (D): now also U9.9 (Q3); no longer U9.19 (Q7)
- net at U10.6 (B): now also U9.5 (Q1); no longer U9.15 (Q5)
- net at U10.7 (C): now also U9.6 (Q2); no longer U9.16 (Q6)
Other:
- moved on the sheet: NIX5, NIX6, R5, R6, U10, U7
