File: pcb_v0/pcb_v0.kicad_sch (KiCad schematic)
At the start: 28 parts, among them J1 Screw_Terminal_01x03, Q1 Q_NMOS_GDS, U1 ATtiny2313-20P, U10 74141, U2 74141, U3 74141, U4 74141, U5 74LS377, U6 74141, U7 74141, U8 74LS377, U9 74LS377

Commit message: save
Connections:
- net at R3.1: now also NIX3.11 (anode); no longer NIX3.10 (anode)
- net at U7.16 (~{Q0}): now also NIX5.10 (cathode0); no longer NIX5.0 (cathode0)
- net at R5.1: now also NIX5.11 (anode); no longer NIX5.10 (anode)
- net at U3.16 (~{Q0}): now also NIX2.10 (cathode0); no longer NIX2.0 (cathode0)
- net at R2.1: now also NIX2.11 (anode); no longer NIX2.10 (anode)
- net at U2.16 (~{Q0}): now also NIX1.10 (cathode0); no longer NIX1.0 (cathode0)
- net at R1.1: now also NIX1.11 (anode); no longer NIX1.10 (anode)
- net at R4.1: now also NIX4.11 (anode); no longer NIX4.10 (anode)
- net at U4.16 (~{Q0}): now also NIX3.10 (cathode0); no longer NIX3.0 (cathode0)
- net at U10.16 (~{Q0}): now also NIX6.10 (cathode0); no longer NIX6.0 (cathode0)
- net at U6.16 (~{Q0}): now also NIX4.10 (cathode0); no longer NIX4.0 (cathode0)
- net at R6.1: now also NIX6.11 (anode); no longer NIX6.10 (anode)
Changed lines of the file:
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@@
     )
     (pin "10")
-    (pin "0")
     (pin "3")
     (pin "1")
@@
     )
     (pin "10")
-    (pin "0")
     (pin "3")
     (pin "1")
@@
     )
     (pin "10")
-    (pin "0")
     (pin "3")
     (pin "1")
@@
     )
     (pin "10")
-    (pin "0")
     (pin "3")
     (pin "1")
@@
     )
     (pin "10")
-    (pin "0")
     (pin "3")
     (pin "1")
@@
     )
     (pin "10")
-    (pin "0")
-    (pin "3")
-    (pin "1")
+    (pin "3")
+    (pin "1")

Commit message: save
Parts:
- removed Q1: Q_NMOS_GDS, Package_TO_SOT_SMD:SOT-223-3_TabPin2, symbol Device:Q_NMOS_GDS
- added Q4: MPSA42, Package_TO_SOT_THT:TO-92_Inline, symbol Transistor_BJT:MPSA42
Connections:
- net GND: now also Q4.1 (E)
- net at R7.1, R8.1: now also Q4.3 (C)

Commit message: save
Parts:
- added R9: R_US, Resistor_THT:R_Axial_DIN0207_L6.3mm_D2.5mm_P7.62mm_Horizontal, symbol Device:R_US
- R1, R2, R3, R4, R5, R6: footprint Resistor_THT:R_Axial_DIN0204_L3.6mm_D1.6mm_P2.54mm_Vertical -> Resistor_THT:R_Axial_DIN0309_L9.0mm_D3.2mm_P12.70mm_Horizontal
- R7, R8: footprint Resistor_THT:R_Axial_DIN0204_L3.6mm_D1.6mm_P2.54mm_Vertical -> Resistor_THT:R_Axial_DIN0207_L6.3mm_D2.5mm_P7.62mm_Horizontal
Connections:
- net hours_en: now reaches U8.11 (CP)
- net hours_en: now also U1.6 (PD2)
- net at Q4.2 (B): now also R9.1
- net minutes_en: now reaches U5.11 (CP)
- net minutes_en: now also U1.3 (PD1)
- net seconds_en: now reaches U9.11 (CP)
- net seconds_en: now also U1.2 (PD0)
- net control_3: now reaches U1.7 (PD3)
- net control_3: now also R9.2
Changed lines of the file:
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@@
 		)
 	)
+	(label "minutes_en"
+		(at 292.1 104.14 0)
+		(effects
+			(font
+				(size 1.27 1.27)
+			)
+			(justify left bottom)
+		)
+	)
+	(label "seconds_en"
+		(at 292.1 101.6 0)
+		(effects
+			(font
+				(size 1.27 1.27)
+			)
+			(justify left bottom)
+		)
+	)
+	(label "minutes_en"
+		(at 350.52 200.66 180)
+		(effects
+			(font
+				(size 1.27 1.27)
+			)
+			(justify right bottom)
+		)
+	)
+	(label "hours_en"
+		(at 350.52 124.46 180)
+		(effects
+			(font
+				(size 1.27 1.27)
+			)
+			(justify right bottom)
+		)
+	)
+	(label "hours_en"
+		(at 292.1 106.68 0)
+		(effects
+			(font
+				(size 1.27 1.27)
+			)
+			(justify left bottom)
+		)
+	)
 	(label "hv"
 		(at 463.55 142.24 0)
@@
 		)
 	)
+	(label "control_3"
+		(at 218.44 171.45 180)
+		(effects
+			(font
+				(size 1.27 1.27)
+			)
+			(justify right bottom)
+		)
+	)
+	(label "control_3"
+		(at 292.1 109.22 0)
+		(effects
+			(font
+				(size 1.27 1.27)
+			)
+			(justify left bottom)
+		)
+	)
 	(label "hv"
 		(at 259.08 144.78 0)
@@
 		)
 	)
+	(label "seconds_en"
+		(at 350.52 276.86 180)
+		(effects
+			(font
+				(size 1.27 1.27)
+			)
+			(justify right bottom)
+		)
+	)
 	(symbol
 		(lib_id "power:+5V")
@@
 			)
 		)
-		(property "Footprint" "Resistor_THT:R_Axial_DIN0204_L3.6mm_D1.6mm_P2.54mm_Vertical"
+		(property "Footprint" "Resistor_THT:R_Axial_DIN0309_L9.0mm_D3.2mm_P12.70mm_Horizontal"
 			(at 459.994 179.324 90)
 			(effects
@@
 	)
 	(symbol
+		(lib_id "Device:R_US")
+		(at 222.25 171.45 270)
+		(unit 1)
+		(exclude_from_sim no)
+		(in_bom yes)
+		(on_board yes)
+		(dnp no)
+		(fields_autoplaced yes)
+		(property "Reference" "R9"
+			(at 222.25 165.1 90)
+			(effects
+				(font
+					(size 1.27 1.27)
+				)
+			)
+		)
+		(property "Value" "R_US"
+			(at 222.25 167.64 90)
+			(effects
+				(font
+					(size 1.27 1.27)
+				)
+			)
+		)
+		(property "Footprint" "Resistor_THT:R_Axial_DIN0207_L6.3mm_D2.5mm_P7.62mm_Horizontal"
+			(at 221.996 172.466 90)
+			(effects
+				(font
+					(size 1.27 1.27)
+				)
+				(hide yes)
+			)
+		)
+		(property "Datasheet" "~"
+			(at 222.25 171.45 0)
+			(effects
+				(font
+					(size 1.27 1.27)
+				)
+				(hide yes)
+			)
+		)
+		(property "Description" ""
+			(at 222.25 171.45 0)
+			(effects
+				(font
+					(size 1.27 1.27)
+				)
+			)
+		)
+		(pin "2"
+		)
+		(pin "1"
+		)
+		(instances
+			(project "pcb_v0"
+				(path "/a1fa5a30-e55c-4a07-9b56-0e31f34de309"
+					(reference "R9")
+					(unit 1)
+				)
+			)
+		)
+	)
+	(symbol
 		(lib_id "nixie_symbols:in-8")
 		(at 443.23 298.45 0)
@@
 			)
 		)
-		(property "Footprint" "Resistor_THT:R_Axial_DIN0204_L3.6mm_D1.6mm_P2.54mm_Vertical"
+		(property "Footprint" "Resistor_THT:R_Axial_DIN0309_L9.0mm_D3.2mm_P12.70mm_Horizontal"
 			(at 459.994 141.224 90)
 			(effects
@@
 			)
 		)
-		(property "Footprint" "Resistor_THT:R_Axial_DIN0204_L3.6mm_D1.6mm_P2.54mm_Vertical"
+		(property "Footprint" "Resistor_THT:R_Axial_DIN0207_L6.3mm_D2.5mm_P7.62mm_Horizontal"
 			(at 232.664 158.496 90)
 			(effects
@@
 			)
 		)
-		(property "Footprint" "Resistor_THT:R_Axial_DIN0204_L3.6mm_D1.6mm_P2.54mm_Vertical"
+		(property "Footprint" "Resistor_THT:R_Axial_DIN0309_L9.0mm_D3.2mm_P12.70mm_Horizontal"
 			(at 459.994 103.124 90)
 			(effects
@@
 			)
 		)
-		(property "Footprint" "Resistor_THT:R_Axial_DIN0204_L3.6mm_D1.6mm_P2.54mm_Vertical"
+		(property "Footprint" "Resistor_THT:R_Axial_DIN0309_L9.0mm_D3.2mm_P12.70mm_Horizontal"
 			(at 459.994 217.424 90)
 			(effects
@@
 			)
 		)
-		(property "Footprint" "Resistor_THT:R_Axial_DIN0204_L3.6mm_D1.6mm_P2.54mm_Vertical"
+		(property "Footprint" "Resistor_THT:R_Axial_DIN0309_L9.0mm_D3.2mm_P12.70mm_Horizontal"
 			(at 459.994 293.624 90)
 			(effects
@@
 			)
 		)
-		(property "Footprint" "Resistor_THT:R_Axial_DIN0204_L3.6mm_D1.6mm_P2.54mm_Vertical"
+		(property "Footprint" "Resistor_THT:R_Axial_DIN0309_L9.0mm_D3.2mm_P12.70mm_Horizontal"
 			(at 459.994 255.524 90)
 			(effects
@@
 			)
 		)
-		(property "Footprint" "Resistor_THT:R_Axial_DIN0204_L3.6mm_D1.6mm_P2.54mm_Vertical"
+		(property "Footprint" "Resistor_THT:R_Axial_DIN0207_L6.3mm_D2.5mm_P7.62mm_Horizontal"
 			(at 258.064 158.496 90)
 			(effects
