File: pcb_v0/pcb_v0.kicad_pcb (KiCad board)
At the start: 2 copper layers, 170 x 50 mm, 28 parts, among them J1 Screw_Terminal_01x03, Q1 Q_NMOS_GDS, U1 ATtiny2313-20P, U10 74141, U2 74141, U3 74141, U4 74141, U5 74LS377, U6 74141, U7 74141, U8 74LS377, U9 74LS377

Commit message: save
Parts:
- moved J1 47.2 mm to (191.5, 52.7), turned to 180 degrees
- moved NE2 1.36 mm to (134.4, 50.0)
- moved NE1 0.50 mm to (84.4, 50.0)
Connections:
- U9 pad 12: Net-(U10-A) -> Net-(U7-A)
- U9 pad 15: Net-(U10-B) -> Net-(U7-B)
- U9 pad 16: Net-(U10-C) -> Net-(U7-C)
- U9 pad 19: Net-(U10-D) -> Net-(U7-D)
- U9 pad 2: Net-(U7-A) -> Net-(U10-A)
- U9 pad 5: Net-(U7-B) -> Net-(U10-B)
- U9 pad 6: Net-(U7-C) -> Net-(U10-C)
- U9 pad 9: Net-(U7-D) -> Net-(U10-D)
Routing:
- net Net-(NIX6-cathode7): track 20.4 -> 0.85 mm
- net Net-(U2-D): track 62.7 -> 67.2 mm
- net Net-(U2-C): track 45.1 -> 48.9 mm
- net Net-(U2-B): track 44.5 -> 46.9 mm
- net Net-(U2-A): track 43.0 -> 44.2 mm
- net Net-(NIX6-cathode1): track 26.7 -> 25.5 mm

Commit message: save
Parts:
- moved R1 4.70 mm to (54.4, 42.4)
- moved U7 4.62 mm to (128.4, 39.8)
- moved U6 3.42 mm to (106.2, 39.8)
- moved U4 2.29 mm to (84.0, 39.8)
- moved U3 1.42 mm to (61.7, 39.8)
- moved J1 0.28 mm to (191.3, 52.5)
Connections:
- NIX1 pad 10: Net-(NIX1-anode) -> Net-(NIX1-cathode0)
- NIX1 pad 11: unconnected-(NIX1-NC-Pad11) -> Net-(NIX1-anode)
- NIX2 pad 10: Net-(NIX2-anode) -> Net-(NIX2-cathode0)
- NIX2 pad 11: unconnected-(NIX2-NC-Pad11) -> Net-(NIX2-anode)
- NIX3 pad 10: Net-(NIX3-anode) -> Net-(NIX3-cathode0)
- NIX3 pad 11: unconnected-(NIX3-NC-Pad11) -> Net-(NIX3-anode)
- NIX4 pad 10: Net-(NIX4-anode) -> Net-(NIX4-cathode0)
- NIX4 pad 11: unconnected-(NIX4-NC-Pad11) -> Net-(NIX4-anode)
- NIX5 pad 10: Net-(NIX5-anode) -> Net-(NIX5-cathode0)
- NIX5 pad 11: unconnected-(NIX5-NC-Pad11) -> Net-(NIX5-anode)
- NIX6 pad 10: Net-(NIX6-anode) -> Net-(NIX6-cathode0)
- NIX6 pad 11: unconnected-(NIX6-NC-Pad11) -> Net-(NIX6-anode)
Routing:
- net Net-(U10-A): track 0.00 -> 50.0 mm
- net Net-(U10-D): track 0.00 -> 36.3 mm
- net Net-(U10-B): track 0.00 -> 35.9 mm
- net Net-(U10-C): track 0.00 -> 32.4 mm
- net Net-(NIX1-cathode0): track 0.00 -> 17.3 mm
- net Net-(U1-PB0): track 97.2 -> 103.9 mm
- net Net-(U1-PB1): track 94.8 -> 95.8 mm
- net Net-(U2-D): track 67.2 -> 66.5 mm
- net Net-(NIX1-anode): track 3.68 -> 4.33 mm
- added copper zone on B.Cu, net (none)
- added copper zone on F.Cu, net (none)

Commit message: save
Parts:
- moved U7 21.1 mm to (148.1, 32.2), turned to -90 degrees
- moved U6 20.5 mm to (125.2, 32.2), turned to -90 degrees
- moved U4 19.9 mm to (102.4, 32.2), turned to -90 degrees
- moved U3 19.3 mm to (79.5, 32.2), turned to -90 degrees
- moved R4 6.17 mm to (124.3, 42.2)
- moved R5 5.47 mm to (154.0, 42.1)
- moved R3 3.49 mm to (105.1, 43.2), turned to -45 degrees
- moved R2 3.48 mm to (76.0, 42.9)
- moved Q1 2.16 mm to (156.3, 34.5)
Routing:
- net Net-(NIX2-cathode5): track 0.00 -> 37.7 mm
- net Net-(NIX4-cathode7): track 0.00 -> 36.0 mm
- net Net-(NIX5-cathode7): track 0.00 -> 32.5 mm
- net Net-(NIX4-cathode6): track 0.00 -> 31.7 mm
- net Net-(NIX5-cathode8): track 0.00 -> 31.5 mm
- net Net-(NIX3-cathode7): track 0.00 -> 31.4 mm
- net Net-(NIX5-cathode9): track 0.00 -> 30.2 mm
- net Net-(NIX2-cathode4): track 0.00 -> 29.2 mm
- net Net-(NIX3-cathode8): track 0.00 -> 26.6 mm
- net Net-(NIX5-cathode2): track 0.00 -> 26.4 mm
- net Net-(NIX5-cathode6): track 0.00 -> 26.3 mm
- net Net-(NIX2-cathode8): track 0.00 -> 24.9 mm
- net Net-(NIX4-cathode8): track 0.00 -> 24.9 mm
- net Net-(NIX3-cathode6): track 0.00 -> 23.1 mm
- net Net-(NIX3-cathode9): track 0.00 -> 23.1 mm
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
Commit message: save
Parts:
- removed Q1: Q_NMOS_GDS, Package_TO_SOT_SMD:SOT-223-3_TabPin2
- added Q4: MPSA42, Package_TO_SOT_THT:TO-92_Inline, F.Cu at (151.3, 33.8)
- added R9: R_US, Resistor_THT:R_Axial_DIN0207_L6.3mm_D2.5mm_P7.62mm_Horizontal, F.Cu at (151.2, 37.8)
- R1, R2, R3, R4, R5, R6: footprint Resistor_THT:R_Axial_DIN0204_L3.6mm_D1.6mm_P2.54mm_Vertical -> Resistor_THT:R_Axial_DIN0309_L9.0mm_D3.2mm_P12.70mm_Horizontal
- R7, R8: footprint Resistor_THT:R_Axial_DIN0204_L3.6mm_D1.6mm_P2.54mm_Vertical -> Resistor_THT:R_Axial_DIN0207_L6.3mm_D2.5mm_P7.62mm_Horizontal
- moved R3 19.9 mm to (90.0, 56.1), turned to 90 degrees
- moved R1 17.0 mm to (56.7, 59.2), turned to 180 degrees
- moved R2 16.0 mm to (60.0, 42.6), turned to -90 degrees
- moved R4 15.1 mm to (130.0, 56.1), turned to 90 degrees
- moved R5 14.5 mm to (160.0, 55.4), turned to 90 degrees
- moved R8 7.52 mm to (139.8, 46.6), turned to -90 degrees
- moved R7 6.10 mm to (80.4, 53.8), turned to 90 degrees
- moved R6 2.92 mm to (175.9, 40.8), turned to 180 degrees
Connections:
- U1 pad 2: unconnected-(U1-PD0-Pad2) -> /seconds_en
- U1 pad 3: unconnected-(U1-PD1-Pad3) -> /minutes_en
- U1 pad 6: unconnected-(U1-PD2-Pad6) -> /hours_en
- U1 pad 7: unconnected-(U1-PD3-Pad7) -> /control_3
- U5 pad 11: unconnected-(U5-CP-Pad11) -> /minutes_en
- U8 pad 11: unconnected-(U8-CP-Pad11) -> /hours_en
- U9 pad 11: unconnected-(U9-CP-Pad11) -> /seconds_en
